Commit message: ROS1 version

File: launch/include/config/robot.urdf.xacro (robot description, xacro)
@@ -9,10 +9,4 @@
     <origin xyz="0 0 0" rpy="0 0 0" />
   </joint>
-  <link name="lidar_link"> </link>
-  <joint name="lidar_joint" type="fixed">
-    <parent link="base_link" />
-    <child link="lidar_link" />
-    <origin xyz="0 0 0" rpy="0 0 0" />
-  </joint>
   <link name="imu_link"> </link>
   <joint name="imu_joint" type="fixed">
@@ -21,8 +15,8 @@
     <origin xyz="0 0 0" rpy="0 0 0" />
   </joint>
-  <link name="rs_helios_top"> </link>
-  <joint name="laser_joint" type="fixed">
-    <parent link="imu_link" />
-    <child link="rs_helios_top" />
+  <link name="velodyne"> </link>
+  <joint name="velodyne_joint" type="fixed">
+    <parent link="chassis_link" />
+    <child link="velodyne" />
     <origin xyz="0 0 0" rpy="0 0 0" />
   </joint>
